Commit message: Release 1.1: Lots of fixes, new CountingVoxelList, new gvl_ompl_planning example and better C++11, Ubuntu 16.04 support
Known issues:
- Octrees are broken on Pascal GPUs
  - confirmed on Titan Xp and GTX 1080 Ti
- the GLM in Ubuntu 16.04 has to be patched to allow usage of the visualizer.
  - see https://github.com/g-truc/glm/issues/530
  - patch for /usr/include/glm/detail/func_common.inl in packages/gpu_voxels/doc/glm_fix_issu530.patch
- Cuda 9.1
  - many incompatibilities are fixed, but there are still failing tests in the voxellist and octree test-suites

API breaking changes:
- GpuVoxels
  - addMap returns null-initialized shared_ptr if map already exists
  - lockSelf, lockBoth & Co removed, replaced by exception-safe lock_guard
  constructs to improve debugging
- TinyXML
  - use system version from APT package libtinyxml-dev

Major changes:
- Changes in CUDA CMake setup
  - uncomment SET(CMAKE_CXX_STANDARD 11) at the top of CMakeLists.txt to activate C++11 mode
  - set -maxrregcount=63 to avoid errors on desktop GPUs with 1024 threads per block
  - always use ICMAKER_CUDA_CPPDEFINES to pass parameters to nvcc
- Added OMPL planning example gvl_ompl_planning  (Thanks to Andreas Hermann)
  - requires C++11
  - incompatible with GPU-Voxels built with PCL 1.7
- Added model "ur10_coarse" voxelized at 9mm
- Added CountingVoxelList to offer pointcloud density filtering  (Thanks to Herbert Pietrzyk)
  - Use remove_underpopulated(minimum_count) to remove outliers
  - Use subtractFromCountingVoxelList to remove the robot and static objects
- Added BitVoxelMap collision with ProbVoxelmap
- ProbVoxelMap
  - insert() parses BitVoxelMeaning to allow freeing single voxels
  - SVCollider checks for noneButEmpty instead of isZero
- Fix CUDA 9 incompatibilities, issue 63
  - version macro
  - cub namespace
  - __ballot vs __ballot_sync

Minor changes:
- DistanceVoxelTest uses double buffering of DistanceVoxelMap to avoid flickering
- ProbVoxelMap: Speed up the clearing of ProbVoxelMap by using memset instead of ctor calls for every voxel
- C++11 fixes
  - icl_core_logging operator<< stringstream bug
  - various fixes collected by dybedal in issue 55
- VoxelList collision
  - added test cases and examples
- fixed memory leaks in TemplateVoxelList
- fixed PCL dependency of examples and helpers, see issue 61
- fix computeLinearLoad returning grid and block size 0
- added many checks after kernel launches to improve error discovery

Other changes:
- Documentation updates

File: packages/gpu_voxels/models/omnirob/omnirob.urdf (robot description, URDF)
Before this commit: robot omniRob, 41 links, 40 joints
Links:
- removed link omnirob_left_lwr_1_link_dummy
- removed link omnirob_left_lwr_2_link_dummy
- removed link omnirob_left_lwr_3_link_dummy
- removed link omnirob_left_lwr_4_link_dummy
- removed link omnirob_left_lwr_5_link_dummy
- removed link omnirob_left_lwr_6_link_dummy
- removed link omnirob_left_lwr_7_link_dummy
- removed link omnirob_right_lwr_1_link_dummy
- removed link omnirob_right_lwr_2_link_dummy
- removed link omnirob_right_lwr_3_link_dummy
- removed link omnirob_right_lwr_4_link_dummy
- removed link omnirob_right_lwr_5_link_dummy
- removed link omnirob_right_lwr_6_link_dummy
- removed link omnirob_right_lwr_7_link_dummy
Joints:
- removed joint omnirob_left_lwr_0_joint_stiffness
- removed joint omnirob_left_lwr_1_joint_stiffness
- removed joint omnirob_left_lwr_2_joint_stiffness
- removed joint omnirob_left_lwr_3_joint_stiffness
- removed joint omnirob_left_lwr_4_joint_stiffness
- removed joint omnirob_left_lwr_5_joint_stiffness
- removed joint omnirob_left_lwr_6_joint_stiffness
- removed joint omnirob_right_lwr_0_joint_stiffness
- removed joint omnirob_right_lwr_1_joint_stiffness
- removed joint omnirob_right_lwr_2_joint_stiffness
- removed joint omnirob_right_lwr_3_joint_stiffness
- removed joint omnirob_right_lwr_4_joint_stiffness
- removed joint omnirob_right_lwr_5_joint_stiffness
- removed joint omnirob_right_lwr_6_joint_stiffness
